File: KiCAD/VCA/VCA.kicad_sch (KiCad schematic)
At the start: 12 parts, among them J1 VIN, J2 VC, J3 VOUT, Q1 J172, Q2 J172, U1 LT1006

Commit message: Notes
Parts:
- R1, R2, R3, R4: value 10k -> ?
- RV1: value Trim Pot -> 100k Trim Pot
- RV2: value Trim Pot -> 1k Trim Pot
Connections:
- net VDD: now also U1.7 (V+); no longer U1.4 (V-)
- net VSS: now also U1.4 (V-); no longer U1.7 (V+)
Other:
- note added: "Is this an error in the original schematic?"
- note added: "What are the resistor values?"
- note added: "Where do the trimpots go?"
- moved on the sheet: R4, RV1, RV2
