File: KiCAD/VCA/_autosave-VCA.kicad_sch (KiCad schematic)
At the start: 14 parts, among them J1 VIN, J2 VC, J3 VOUT, Q1 J172, Q2 J172, U1 LT1006

Commit message: VCA Schematic
Parts:
- R1, R2, R3, R4: value ? -> 10k
Connections:
- net VDD: now also C1.1; no longer C1.2
- net VSS: now also C1.2
- net at Q1.1 (D), R1.2, R3.1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: no longer C1.1
Other:
- note removed: "Is this an error in the original schematic?"
- note removed: "What are the resistor values?"
- moved on the sheet: C1, J1, J2, J3, Q1, Q2, R1, R3, R4, R5, RV1, RV2
