File: KiCAD/Power/Power.kicad_pcb (KiCad board)
At the start: 2 copper layers, 18 parts, among them J1 Barrel_Jack_Switch_MountingPin, J2 Conn_01x03_Pin, U1 LM317L_SOT-89, U2 LM337_SOT223, U3 LM336Z-2.5v

Commit message: MidMount Capacitors
Parts:
- C1, C2, C3: footprint Capacitor_THT:CP_Radial_D10.0mm_P5.00mm -> HackSynth:CP_Radial_D10.0mm_P5.00mm_MidMount
- U1: value LM317L_SOT-89 -> LM317 TO-220; footprint HackSynth:LM317 - TO-220-3_Vertical -> HackSynth:LM317 - TO-220-3_Horizontal_TabDown
- U2: value LM337_SOT223 -> LM337 TO-220; footprint HackSynth:LM337 - TO-220-3_Vertical -> HackSynth:LM337 - TO-220-3_Horizontal_TabDown
- U3: footprint HackSynth:TO-92_Inline - Handsolder -> Package_TO_SOT_THT:TO-92_Inline
- moved U3 61.5 mm to (137.7, 52.9)
- moved R1 40.9 mm to (128.2, 63.2)
- moved R2 40.9 mm to (128.2, 67.2)
- moved R3 40.9 mm to (128.2, 71.3)
- moved R4 40.9 mm to (128.2, 75.3)
- moved D1 40.9 mm to (117.3, 63.3)
- moved D2 40.9 mm to (117.3, 67.5)
- moved D3 40.9 mm to (117.3, 71.8)
- moved D4 40.9 mm to (117.3, 76.0)
- moved J1 39.6 mm to (137.0, 38.3)
- moved J2 39.6 mm to (128.7, 52.0)
- moved C4 38.1 mm to (139.5, 64.5)
- moved C5 38.1 mm to (139.5, 71.0)
- moved C3 37.6 mm to (117.4, 58.1)
- moved C2 27.9 mm to (105.9, 58.1)
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Other:
- board outline added: 65 x 60 mm

Commit message: Power PCB
Parts:
- U3: footprint Package_TO_SOT_THT:TO-92_Inline -> HackSynth:TO-92_Inline - Handsolder
- moved J2 112.2 mm to (109.0, 162.5)
- moved C4 88.5 mm to (108.5, 147.4)
- moved C5 88.5 mm to (94.8, 147.4)
- moved R3 75.8 mm to (96.1, 140.0), turned to 90 degrees
- moved D1 73.7 mm to (91.5, 132.4), turned to -90 degrees
- moved D2 64.9 mm to (114.5, 132.4), turned to -90 degrees
- moved D3 62.8 mm to (100.7, 132.4), turned to -90 degrees
- moved R4 59.9 mm to (109.9, 132.4), turned to -90 degrees
- moved U3 59.7 mm to (104.3, 102.4), turned to 180 degrees
- moved D4 57.6 mm to (105.3, 132.4), turned to -90 degrees
- moved R1 54.6 mm to (90.2, 102.4)
- moved U1 45.3 mm to (97.0, 127.0)
- moved U2 45.3 mm to (109.1, 127.0)
- moved R2 40.4 mm to (108.2, 102.4)
- moved J1 39.5 mm to (98.3, 46.3), turned to 180 degrees
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Routing:
- added copper zone on B.Cu, net GND
- added copper zone on F.Cu, net GND
- added copper zone on In1.Cu, net GND
- added copper zone on In2.Cu, net GND
Other:
- board size 65 x 60 mm -> 30 x 132.6 mm
- copper layers 2 -> 4

Commit message: Power PCB
Parts:
- added G***: LOGO, CCHS:PancakeLegend_Logo_SolderMask, B.Cu at (115.2, 126.5)
- added REF**: Symbol_Barrel_Polarity, Symbol:Symbol_Barrel_Polarity, F.Cu at (108.1, 44.6)
- added REF**: CCHS_Logo_Small_NoText, CCHS:CCHS_Logo_Small_NoText, B.Cu at (107.8, 53.0)
- C4, C5: footprint Capacitor_THT:CP_Radial_D5.0mm_P2.50mm -> HackSynth:CP_Radial_D5.2mm_P2.50mm_LayDown
- moved C5 37.0 mm to (118.2, 118.6), turned to 180 degrees
- moved J2 29.2 mm to (120.2, 135.6)
- moved C4 29.0 mm to (112.2, 118.6), turned to 180 degrees
- moved R4 26.2 mm to (127.2, 112.6)
- moved D4 21.9 mm to (127.2, 130.6), turned to 90 degrees
- moved R3 21.0 mm to (103.2, 120.3)
- moved J1 19.0 mm to (117.0, 50.0)
- moved U2 18.1 mm to (121.3, 113.7)
- moved U1 18.1 mm to (109.2, 113.7)
- moved R1 17.6 mm to (102.4, 89.6)
- moved R2 17.6 mm to (120.4, 89.6)
- moved U3 17.6 mm to (116.5, 89.6)
- moved C3 16.7 mm to (125.9, 83.8)
- moved C2 16.0 mm to (125.9, 72.3)
- moved D1 15.7 mm to (107.2, 130.6), turned to 90 degrees
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Connections:
- net Net-(D3-K) renamed VDD
- net Net-(D4-A) renamed VSS
Routing:
- net Net-(D2-A): track 0.00 -> 62.8 mm
- net Net-(D2-K): track 0.00 -> 22.1 mm
- net Net-(D1-A): track 0.00 -> 17.3 mm
- added copper zone on In2.Cu, net Net-(D1-K)
- added copper zone on F.Cu, net VDD
- added copper zone on B.Cu, net VSS
- removed copper zone on B.Cu, net GND
- removed copper zone on F.Cu, net GND
- removed copper zone on In2.Cu, net GND
Other:
- board size 30 x 132.6 mm -> 30 x 102 mm
- board text added: "+/-12v"
- board text added: "DC 24v"
- board text added: "POWER v1-0"

Commit message: Power PCB
Parts:
- removed G***: LOGO, CCHS:PancakeLegend_Logo_SolderMask
- removed the REF** at (107.8, 53.0)
- added Ref**: Val**, HackSynth:PancakeLegend Logo - 10mm, B.Cu at (121.2, 105.5)
- added Ref**: Val**, HackSynth:CCHS Logo - 10mm, B.Cu at (109.2, 105.6)
- moved J2 1.37 mm to (120.2, 134.2)
- moved C1 0.83 mm to (126.2, 61.5)
- moved C2 0.83 mm to (126.2, 73.0)
- moved C3 0.83 mm to (126.2, 84.5)
- moved C4 0.64 mm to (112.2, 118.0)
- moved C5 0.64 mm to (118.2, 118.0)
- moved J1 0.61 mm to (117.0, 50.6)
- moved R1 0.61 mm to (102.4, 90.2)
- moved R2 0.61 mm to (120.4, 90.2)
- moved REF** 0.61 mm to (108.1, 45.2)
- moved U3 0.61 mm to (116.5, 90.2)
Routing:
- net Net-(D2-A): track 62.8 -> 61.3 mm
Other:
- board size 30 x 102 mm -> 30 x 100 mm
- board text added: "POWER v1-0 - PancakeLegend 2025"
- board text removed: "POWER v1-0"

Commit message: Power PCB Gerbers
Parts:
- added D5: LED, HackSynth:LED_D5.0mm, F.Cu at (104.8, 47.0)
- added R5: 1.1k, Resistor_THT:R_Axial_DIN0207_L6.3mm_D2.5mm_P7.62mm_Horizontal, F.Cu at (112.5, 50.8)
- REF**: moved to B.Cu
- moved REF** 2.58 mm to (106.0, 43.8), turned to 180 degrees
- moved R2 0.20 mm to (120.2, 90.2)
Routing:
- net Net-(D1-K): track 0.00 -> 79.5 mm
- net Net-(D2-A): track 61.3 -> 36.1 mm
- net Net-(D5-K): track 0.00 -> 9.62 mm
- net Net-(D1-A): track 17.3 -> 18.1 mm
- added copper zone on B.Cu, net GND
- added copper zone on F.Cu, net GND
- added copper zone on In1.Cu, net VDD
- added copper zone on In2.Cu, net VSS
- removed copper zone on In1.Cu, net GND
- removed copper zone on In2.Cu, net Net-(D1-K)
- removed copper zone on F.Cu, net VDD
- removed copper zone on B.Cu, net VSS

Commit message: Power PCB Cleanup
Parts:
- moved C1 0.50 mm to (126.2, 61.0)
- moved C2 0.50 mm to (126.2, 72.5)
- moved C3 0.50 mm to (126.2, 84.0)
- moved C4 0.50 mm to (112.2, 117.5)
- moved C5 0.50 mm to (118.2, 117.5)
- moved D1 0.50 mm to (107.2, 130.1)
- moved D2 0.50 mm to (123.2, 130.1)
- moved D3 0.50 mm to (103.2, 130.1)
- moved D4 0.50 mm to (127.2, 130.1)
- moved D5 0.50 mm to (104.8, 46.5)
- moved J1 0.50 mm to (117.0, 50.1)
- moved J2 0.50 mm to (120.2, 133.7)
- moved R1 0.50 mm to (102.4, 89.8)
- moved R2 0.50 mm to (120.2, 89.8)
- moved R3 0.50 mm to (103.2, 119.8)
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