File: KiCAD/Mixer/Mixer.kicad_pcb (KiCad board)
At the start: 2 copper layers, 30 x 100 mm, 24 parts, among them J1 IN_1, J2 IN_2, J3 OUT, J5 Conn_01x03, J6 Conn_01x03, Q1 BC547, U1 TL072

Commit message: Mixer PCB - Gerbers
Parts:
- moved Ref** 55.8 mm to (150.0, 112.8)
- moved Ref** 52.0 mm to (150.0, 125.0)
- moved C2 14.5 mm to (162.5, 89.5)
- moved R3 2.06 mm to (138.0, 78.1)
- moved R4 2.06 mm to (142.0, 85.8)
- moved R5 2.00 mm to (158.0, 78.2)
- moved R6 2.00 mm to (162.0, 85.8)
- moved Q1 1.69 mm to (148.7, 84.7)
- moved C1 1.50 mm to (152.5, 89.5)
- moved R1 1.00 mm to (138.0, 100.8)
- moved R2 1.00 mm to (142.0, 100.8)
- moved R7 1.00 mm to (158.0, 100.8)
- moved R8 1.00 mm to (162.0, 93.2)
- moved U1 1.00 mm to (150.0, 97.0)
- moved C3 0.50 mm to (147.5, 104.5)
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Connections:
- J3 pad G: Net-(J3-PadG) -> GND
- J3 pad S: Net-(J3-PadG) -> GND
Routing:
- net Net-(J3-PadT): track 33.1 -> 41.5 mm
- net Net-(Q1-E): track 12.8 -> 18.1 mm
- net Net-(U1A--): track 22.9 -> 26.0 mm
- net Net-(R3-Pad1): track 9.85 -> 7.79 mm
- net Net-(U1B--): track 19.2 -> 20.4 mm
- net Net-(R2-Pad1): track 34.4 -> 33.2 mm
- net Net-(R1-Pad1): track 29.4 -> 28.2 mm
- net NOISE: track 48.1 -> 47.2 mm
- net VSS: track 81.1 -> 80.3 mm
Other:
- board text added: "OUT"
