File: KiCAD/MIDI_to_CV/MIDI_to_CV.kicad_pcb (KiCad board)
At the start: 2 copper layers, 30 x 100 mm, 21 parts, among them J1 DIN-5_180degree, J2 PITCH, J3 GATE, J4 Conn_01x03_Socket, J5 Conn_01x03_Socket, U1 ATtiny45-20P, U2 6N138, U3 L7805

Commit message: Footprint Edits
Changed lines of the file:
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@@
 		(tags "THT DIP DIL PDIP 2.54mm 7.62mm 300mil LongPads")
 		(property "Reference" "U2"
-			(at 0.065 0.07 0)
+			(at 0.065 5.94 0)
 			(layer "F.SilkS")
 			(effects
@@
 		(tags "THT DIP DIL PDIP 2.54mm 7.62mm 300mil LongPads")
 		(property "Reference" "U1"
-			(at 0.065 0.07 0)
-			(layer "F.SilkS")
-			(effects
+			(at 0 6 0)
+			(layer "F.SilkS")
+			(effects
