File: KiCAD/MIDI_to_CV/MIDI_to_CV.kicad_sch (KiCad schematic)
At the start: 18 parts, among them J1 GATE, J2 DIN-5_180degree, J3 PITCH, J4 Conn_01x03_Socket, J5 Conn_01x03_Socket, U1 ATtiny45-20P, U2 6N138, U3 L7805

Commit message: MIDI to CV - PCB Placement
Parts:
- C2: value 470uF -> 10uF 10v; footprint HackSynth:CP_Radial_D10.0mm_P5.00mm_MidMount -> HackSynth:CP_Radial_D5.2mm_P2.50mm_LayDown
- C3: value 1uF -> 1uF 10v
Other:
- note removed: "Cap Oversized??"

Commit message: MIDI to CV - PCB
Parts:
- J1: renamed from J2; footprint HackSynth:DIN-5 MIDI Jack -> HackSynth:DIN-5 - DS-5-07A - MIDI Jack
- renumbered J1 to J2, J5 to J4, J4 to J5
Other:
- moved on the sheet: J4, J5

Commit message: MIDI to CV - Gerbers
Parts:
- C2: value 10uF 10v -> 10uF 25v
- C3: value 1uF 10v -> 1uF 50v
- J2: value GATE -> PITCH
- J3: value PITCH -> GATE
Connections:
- net GND: now also J1.2
- no-connect marks 6 -> 5
Other:
- moved on the sheet: J4, J5

Commit message: MIDI to CV Cap Footprint Change
Parts:
- C2, C3: footprint HackSynth:CP_Radial_D5.2mm_P2.50mm_LayDown -> HackSynth:CP_Radial_D4.0mm_P1.50mm
Changed lines of the file:
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@@
 			)
 		)
-		(property "Footprint" "HackSynth:CP_Radial_D5.2mm_P2.50mm_LayDown"
+		(property "Footprint" "HackSynth:CP_Radial_D4.0mm_P1.50mm"
 			(at 121.6152 160.02 0)
 			(effects
@@
 			)
 		)
-		(property "Footprint" "HackSynth:CP_Radial_D5.2mm_P2.50mm_LayDown"
+		(property "Footprint" "HackSynth:CP_Radial_D4.0mm_P1.50mm"
 			(at 148.2852 160.02 0)
 			(effects

Commit message: Backup Cleanup
Changed lines of the file:
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@@
 		(dnp no)
 		(property "Reference" "R3"
-			(at 161.036 49.53 0)
+			(at 161.544 49.784 0)
 			(effects
 				(font
@@
 		)
 		(property "Value" "4.7k"
-			(at 161.036 52.07 0)
+			(at 161.544 51.562 0)
 			(effects
 				(font
@@
 		(on_board yes)
 		(dnp no)
-		(fields_autoplaced yes)
 		(property "Reference" "R2"
-			(at 172.72 31.7499 0)
+			(at 172.466 32.258 0)
 			(effects
 				(font
@@
 		)
 		(property "Value" "220R"
-			(at 172.72 34.2899 0)
+			(at 172.466 34.0359 0)
 			(effects
 				(font
@@
 		(on_board yes)
 		(dnp no)
-		(fields_autoplaced yes)
 		(property "Reference" "R4"
-			(at 132.08 83.82 90)
+			(at 132.08 87.884 90)
 			(effects
 				(font
@@
 		)
 		(property "Value" "1k"
-			(at 132.08 86.36 90)
+			(at 132.08 90.17 90)
 			(effects
 				(font
@@
 		(on_board yes)
 		(dnp no)
-		(fields_autoplaced yes)
 		(property "Reference" "R1"
-			(at 127 29.21 90)
+			(at 127 33.274 90)
 			(effects
 				(font
@@
 		)
 		(property "Value" "220R"
-			(at 127 31.75 90)
+			(at 127 35.56 90)
 			(effects
 				(font
@@
 		(dnp no)
 		(property "Reference" "R5"
-			(at 139.7 96.012 90)
+			(at 139.7 94.996 90)
 			(effects
 				(font
@@
 		)
 		(property "Value" "1k"
-			(at 139.7 98.552 90)
-			(effects
-				(font
+			(at 139.7 92.71 90)
+			(effects
+				(font

Commit message: Footprint Edits
Parts:
- added G1: ~, symbol HackSynth:CCHS_Logo
- added G2: ~, symbol HackSynth:Logo_PancakeLegend
Changed lines of the file:
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@@
+	)
+	(symbol
+		(lib_id "HackSynth:CCHS_Logo")
+		(at 276.86 172.72 0)
+		(unit 1)
+		(exclude_from_sim no)
+		(in_bom yes)
+		(on_board yes)
+		(dnp no)
+		(fields_autoplaced yes)
+		(property "Reference" "G1"
+			(at 276.86 180.34 0)
+			(effects
+				(font
+					(size 1.27 1.27)
+				)
+				(hide yes)
+			)
+		)
+		(property "Value" "~"
+			(at 283.21 173.89 0)
+			(effects
+				(font
+					(size 1.27 1.27)
+				)
+				(justify left)
+			)
+		)
+		(property "Footprint" ""
+			(at 276.86 172.72 0)
+			(effects
+				(font
+					(size 1.27 1.27)
+				)
+				(hide yes)
+			)
+		)
+		(property "Datasheet" ""
+			(at 276.86 172.72 0)
+			(effects
+				(font
+					(size 1.27 1.27)
+				)
+				(hide yes)
+			)
+		)
+		(property "Description" ""
+			(at 276.86 172.72 0)
+			(effects
+				(font
+					(size 1.27 1.27)
+				)
+				(hide yes)
+			)
+		)
+		(instances
+			(project "MIDI_to_CV"
+				(path "/e50e7ffb-93d3-426c-8afd-d373aea943b3"
+					(reference "G1")
+					(unit 1)
+				)
+			)
+		)
 	)
 	(symbol
@@
 					(unit 1)
 				)
+			)
+		)
+	)
+	(symbol
+		(lib_id "HackSynth:Logo_PancakeLegend")
+		(at 264.16 173.355 0)
+		(unit 1)
+		(exclude_from_sim no)
+		(in_bom yes)
+		(on_board yes)
+		(dnp no)
+		(fields_autoplaced yes)
+		(property "Reference" "G2"
+			(at 264.16 180.975 0)
+			(effects
+				(font
+					(size 1.27 1.27)
+				)
+				(hide yes)
+			)
+		)
+		(property "Value" "~"
+			(at 270.51 173.2549 0)
+			(effects
+				(font
+					(size 1.27 1.27)
+				)
+				(justify left)
+			)
+		)
+		(property "Footprint" ""
+			(at 264.16 173.355 0)
+			(effects
+				(font
+					(size 1.27 1.27)
+				)
+				(hide yes)
+			)
+		)
+		(property "Datasheet" ""
+			(at 264.16 173.355 0)
+			(effects
+				(font
+					(size 1.27 1.27)
+				)
+				(hide yes)
+			)
+		)
+		(property "Description" ""
+			(at 264.16 173.355 0)
+			(effects
+				(font
+					(size 1.27 1.27)
+				)
+				(hide yes)
+			)
+		)
+		(instances
+			(project "MIDI_to_CV"
+				(path "/e50e7ffb-93d3-426c-8afd-d373aea943b3"
+					(reference "G2")
+					(unit 1)
+				)
