File: KiCAD/Chorus/Chorus.kicad_pcb (KiCad board)
At the start: 2 copper layers, 50 x 100 mm, 87 parts, among them J1 IN, J2 OUT, J3 Conn_01x03, J4 Conn_01x03, Q1 BC337, Q2 BC337, SW1 SW_SPDT, U1 TL072, U2 TL072, U4 L7805, U5 TL072, U6 PT2399

Commit message: Chorus PCB Start
Parts:
- removed U6: PT2399, HackSynth:DIP-16_W7.62mm_LongPads
- added U3: TL072, HackSynth:DIP-8_W7.62mm_LongPads, F.Cu at (150.0, 110.6)
- U4: value L7805 -> PT2399; footprint HackSynth:L7805 - TO-220-3_Horizontal_TabDown -> HackSynth:DIP-16_W7.62mm_LongPads
- U5: value TL072 -> L7805; footprint HackSynth:DIP-8_W7.62mm_LongPads -> HackSynth:L7805 - TO-220-3_Horizontal_TabDown
- moved G1 100.6 mm to (156.8, 139.5)
- moved G2 99.9 mm to (143.5, 139.2)
- moved C3 70.7 mm to (153.4, 51.3), turned to -90 degrees
- moved R3 68.4 mm to (168.8, 53.5), turned to -90 degrees
- moved R4 68.3 mm to (165.8, 53.5), turned to -90 degrees
- moved J2 66.2 mm to (165.0, 62.5), turned to 90 degrees
- moved C8 65.6 mm to (162.2, 82.2), turned to 180 degrees
- moved C5 65.1 mm to (162.2, 74.9), turned to 180 degrees
- moved J1 65.1 mm to (135.0, 62.5), turned to -90 degrees
- moved C24 64.7 mm to (159.4, 146.8)
- moved C4 64.7 mm to (162.2, 71.5), turned to 180 degrees
- moved U1 64.3 mm to (150.0, 63.2)
- moved C23 64.0 mm to (159.4, 140.2)
- moved C6 61.9 mm to (157.2, 78.2)
- moved C2 61.3 mm to (150.0, 56.3), turned to 90 degrees
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Connections:
- C25 pad 1: Net-(U5A--) -> Net-(U3A--)
- C28 pad 1: Net-(U6-REF) -> Net-(U4-REF)
- C29 pad 1: Net-(U6-CC1) -> Net-(U4-CC1)
- C30 pad 1: Net-(U6-CC0) -> Net-(U4-CC0)
- C31 pad 1: Net-(U6-LPF1-IN) -> Net-(U4-LPF1-IN)
- C31 pad 2: Net-(U6-LPF1-OUT) -> Net-(U4-LPF1-OUT)
- C32 pad 2: Net-(U6-LPF2-IN) -> Net-(U4-LPF2-IN)
- C33 pad 1: Net-(U6-OP2-OUT) -> Net-(U4-OP2-OUT)
- C33 pad 2: Net-(U6-OP2-IN) -> Net-(U4-OP2-IN)
- C34 pad 1: Net-(U6-OP1-IN) -> Net-(U4-OP1-IN)
- C34 pad 2: Net-(U6-OP1-OUT) -> Net-(U4-OP1-OUT)
- R26 pad 1: Net-(U5A--) -> Net-(U3A--)
- R26 pad 2: Net-(U5B-+) -> Net-(U3B-+)
- R27 pad 1: Net-(U5A-+) -> Net-(U3A-+)
- R28 pad 2: Net-(U5A-+) -> Net-(U3A-+)
- R30 pad 2: Net-(U6-LPF1-IN) -> Net-(U4-LPF1-IN)
- R31 pad 1: Net-(U6-LPF1-OUT) -> Net-(U4-LPF1-OUT)
- R33 pad 1: Net-(U6-LPF2-IN) -> Net-(U4-LPF2-IN)
- R34 pad 1: Net-(U6-OP2-OUT) -> Net-(U4-OP2-OUT)
- R36 pad 2: Net-(U5B--) -> Net-(U3B--)
- RV4 pad 1: Net-(U5B-+) -> Net-(U3B-+)
- RV4 pad 2: Net-(U5B-+) -> Net-(U3B-+)
- U4 pad 1: Net-(D5-K) -> +5V
- U4 pad 2: GND -> Net-(U4-REF)
- U4 pad 3: +5V -> GND
- U5 pad 1: Net-(R27-Pad2) -> Net-(D5-K)
- U5 pad 2: Net-(U5A--) -> GND
- U5 pad 3: Net-(U5A-+) -> +5V
Routing:
- added copper zone on F.Cu, net GND
- added copper zone on B.Cu, net VDD

Commit message: Chorus Trace Begin
Parts:
- removed R35, R36, R38, R39: 10k, HackSynth:R_Vertical_P2.54mm
- removed R37: 4.7k, HackSynth:R_Vertical_P2.54mm
- removed R40: 100k, HackSynth:R_Vertical_P2.54mm
- added R18: 10k, HackSynth:R_Vertical_P2.54mm, F.Cu at (143.1, 122.5)
- added R19: 100k, HackSynth:R_Vertical_P2.54mm, F.Cu at (143.1, 125.2)
- added R20: 56k, HackSynth:R_Vertical_P2.54mm, F.Cu at (156.9, 125.2)
- added R21: 10k, HackSynth:R_Vertical_P2.54mm, F.Cu at (156.9, 119.8)
- added R22: 4.7k, HackSynth:R_Vertical_P2.54mm, F.Cu at (156.9, 122.5)
- added R23: 100k, HackSynth:R_Vertical_P2.54mm, F.Cu at (134.5, 106.1)
- R27: value 100k -> 10k
- R28: value 56k -> 10k
- moved R28 45.4 mm to (173.5, 88.6), turned to 90 degrees
- moved R29 36.6 mm to (168.0, 97.4)
- moved R26 35.6 mm to (165.2, 97.4), turned to 90 degrees
- moved C21 22.2 mm to (162.2, 92.8)
- moved C22 20.7 mm to (162.2, 105.8), turned to 180 degrees
- moved R15 16.5 mm to (165.2, 88.6)
- moved R27 14.9 mm to (143.1, 119.8), turned to 0 degrees
- moved R12 14.8 mm to (173.5, 74.1)
- moved C4 9.65 mm to (162.2, 70.0), turned to 180 degrees
- moved C18 6.33 mm to (157.2, 89.5)
- moved C14 6.18 mm to (157.2, 86.2)
- moved C13 6.04 mm to (157.2, 83.0)
- moved R17 5.75 mm to (170.8, 88.6)
- moved C9 5.01 mm to (137.7, 76.8), turned to 0 degrees
- moved C10 5.00 mm to (137.7, 80.0), turned to 0 degrees
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- renumbered C37 to C12, C35 to C13, C31 to C14, C34 to C15, C25 to C16, C33 to C17, C32 to C18, C26 to C19, C29 to C20, C36 to C21, C38 to C22, C30 to C25, C6 to C4, C4 to C5, C5 to C6, D6 to D5, D5 to D6, RV4 to RV3, RV5 to RV4
Connections:
- C13 pad 1: Net-(C35-Pad1) -> Net-(C13-Pad1)
- C13 pad 2: Net-(C35-Pad2) -> Net-(C13-Pad2)
- C21 pad 1: Net-(C35-Pad2) -> Net-(C13-Pad2)
- C3 pad 1: Net-(C3-Pad1) -> Net-(U1B--)
- C3 pad 2: Net-(U1B--) -> Net-(C3-Pad2)
- C39 pad 1: Net-(D6-A) -> Net-(D5-A)
- D5 pad 2: Net-(D6-A) -> Net-(D5-A)
- Q1 pad 2: Net-(D6-A) -> Net-(D5-A)
- R2 pad 1: Net-(U1B--) -> Net-(C1-Pad1)
- R2 pad 2: Net-(C1-Pad1) -> Net-(U1B--)
- R26 pad 1: Net-(U3A--) -> D IN
- R26 pad 2: Net-(U3B-+) -> Net-(C13-Pad1)
- R27 pad 1: Net-(U3A-+) -> Net-(SW1-A)
- R27 pad 2: Net-(R27-Pad2) -> Net-(SW1-B)
- R28 pad 1: GND -> D OUT
- R28 pad 2: Net-(U3A-+) -> D IN
- R29 pad 1: +5V -> Net-(SW1-B)
- R29 pad 2: Net-(D6-A) -> Net-(C13-Pad2)
- R3 pad 1: DELAY -> Net-(U1B--)
- R3 pad 2: Net-(U1B--) -> DELAY
- R30 pad 1: Net-(C35-Pad2) -> Net-(C13-Pad2)
- R31 pad 2: Net-(C35-Pad2) -> Net-(C13-Pad2)
- R4 pad 2: Net-(C3-Pad1) -> Net-(C3-Pad2)
- R6 pad 1: Net-(U1A--) -> Net-(C2-Pad1)
- R6 pad 2: Net-(C2-Pad1) -> Net-(U1A--)
- R7 pad 1: Net-(C3-Pad1) -> Net-(C3-Pad2)
- R8 pad 1: Net-(D1-A) -> Net-(C2-Pad1)
- R8 pad 2: Net-(C2-Pad1) -> Net-(D1-A)
- RV3 pad 3: Net-(R27-Pad2) -> Net-(R19-Pad2)
- U1 pad 7: Net-(C3-Pad1) -> Net-(C3-Pad2)
- U3 pad 1: Net-(R27-Pad2) -> Net-(R19-Pad2)
Routing:
- net VDD: track 0.00 -> 152.3 mm, vias 0 -> 4
- net FEEDBACK: track 0.00 -> 94.2 mm, vias 0 -> 2
- net Net-(U1B--): track 0.00 -> 63.7 mm, vias 0 -> 1
- net Net-(U1A--): track 0.00 -> 55.0 mm
- net Net-(D1-A): track 0.00 -> 54.9 mm
- net Net-(C3-Pad2): track 0.00 -> 32.6 mm
- net Net-(U2A-+): track 0.00 -> 27.9 mm
- net Net-(C1-Pad1): track 0.00 -> 21.9 mm
- net Net-(C2-Pad1): track 0.00 -> 21.6 mm
- net Net-(J2-PadT): track 0.00 -> 15.9 mm
- net Net-(C8-Pad1): track 0.00 -> 15.8 mm
- net D OUT: track 0.00 -> 15.6 mm
- net Net-(C6-Pad1): track 0.00 -> 12.7 mm
- net Net-(C1-Pad2): track 0.00 -> 10.7 mm
- net D IN: track 0.00 -> 9.53 mm
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
Commit message: Chorus Trace v1
Parts:
- moved G1 72.0 mm to (134.6, 71.0)
- moved U5 18.8 mm to (150.0, 129.2), turned to 180 degrees
- moved C24 18.5 mm to (141.0, 144.5), turned to 180 degrees
- moved G2 12.0 mm to (155.3, 136.9)
- moved C27 10.2 mm to (142.8, 138.8), turned to 90 degrees
- moved C23 4.27 mm to (159.0, 144.5), turned to 180 degrees
- moved R33 2.75 mm to (170.8, 106.1)
- moved R34 2.75 mm to (168.0, 106.1)
- turned C7 to 180 degrees
Connections:
- C8 pad 1: Net-(C8-Pad1) -> GND
- C8 pad 2: GND -> Net-(C8-Pad2)
- R12 pad 2: Net-(C8-Pad1) -> Net-(C8-Pad2)
- R13 pad 1: Net-(C8-Pad1) -> Net-(C8-Pad2)
- R16 pad 1: Net-(U2B--) -> GND
- R16 pad 2: GND -> Net-(U2B--)
- R19 pad 1: Net-(U3A-+) -> Net-(R19-Pad1)
- R19 pad 2: Net-(R19-Pad2) -> Net-(U3A-+)
- R22 pad 1: GND -> Net-(R22-Pad1)
- R22 pad 2: Net-(R22-Pad2) -> GND
- R27 pad 1: Net-(SW1-A) -> Net-(SW1-B)
- R27 pad 2: Net-(SW1-B) -> Net-(SW1-A)
- R31 pad 1: Net-(U4-LPF1-OUT) -> Net-(C13-Pad2)
- R31 pad 2: Net-(C13-Pad2) -> Net-(U4-LPF1-OUT)
- R32 pad 1: Net-(SW1-B) -> Net-(C19-Pad1)
- R32 pad 2: Net-(C19-Pad1) -> Net-(SW1-B)
- R33 pad 1: Net-(U4-LPF2-IN) -> Net-(C19-Pad1)
- R33 pad 2: Net-(C19-Pad1) -> Net-(U4-LPF2-IN)
- R34 pad 1: Net-(U4-OP2-OUT) -> Net-(C19-Pad1)
- R34 pad 2: Net-(C19-Pad1) -> Net-(U4-OP2-OUT)
- RV3 pad 3: Net-(R19-Pad2) -> Net-(R19-Pad1)
- RV4 pad 3: Net-(R22-Pad2) -> Net-(R22-Pad1)
- U3 pad 1: Net-(R19-Pad2) -> Net-(R19-Pad1)
Routing:
- net VDD: track 152.3 -> 8.22 mm
- net VSS: track 0.00 -> 131.2 mm
- net +5V: track 0.00 -> 103.2 mm, vias 0 -> 2
- net Net-(R15-Pad2): track 0.00 -> 100.7 mm, vias 0 -> 2
- net Net-(Q2-B): track 0.00 -> 65.5 mm, vias 0 -> 1
- net DELAY: track 0.00 -> 64.6 mm
- net Net-(SW1-B): track 0.00 -> 61.0 mm
- net Net-(C8-Pad2): track 0.00 -> 50.7 mm, vias 0 -> 2
- net Net-(R19-Pad1): track 0.00 -> 41.1 mm, vias 0 -> 1
- net Net-(U3B-+): track 0.00 -> 40.5 mm, vias 0 -> 1
- net Net-(U2B-+): track 0.00 -> 40.2 mm, vias 0 -> 1
- net Net-(U2A--): track 0.00 -> 38.8 mm, vias 0 -> 2
- net Net-(D5-A): track 0.00 -> 36.8 mm
- net TIME: track 0.00 -> 34.0 mm
- net Net-(U4-LPF2-IN): track 0.00 -> 30.8 mm, vias 0 -> 1
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
Commit message: Chorus Legends
Parts:
- renumbered C39 to C26
Routing:
- net GND: track 17.1 -> 13.0 mm
Other:
- board text added: "DECAY"
- board text added: "DEPTH"
- board text added: "FEED"
- board text added: "IN"
- board text added: "OUT"
- board text added: "RATE"
Changed lines of the file:
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@@
 		(tags "WQP-PJ398SM WQP-PJ301M-12 TRS 3.5mm mono vertical jack thonkiconn qingpu")
 		(property "Reference" "J2"
-			(at 3.25 5.75 90)
+			(at -3.34 5.82 90)
 			(layer "F.SilkS")
 			(effects
@@
 		)
 		(property "Value" "TL072"
-			(at 0 6.14 0)
+			(at 0.025 3.91 0)
 			(layer "F.Fab")
 			(effects
@@
 		)
 		(property "Value" "TL072"
-			(at 0 6.14 0)
+			(at 0 3.915 0)
 			(layer "F.Fab")
 			(effects
@@
 		(descr "CP, Radial series, Radial, pin pitch=5.00mm, diameter=10mm, height=16mm, Electrolytic Capacitor")
 		(tags "CP Radial series Radial pin pitch 5.00mm diameter 10mm height 16mm Electrolytic Capacitor")
-		(property "Reference" "C39"
+		(property "Reference" "C26"
 			(at 0 -14.5 90)
 			(layer "F.SilkS")
@@
 		)
 		(property "Value" "TL072"
-			(at 0 6.14 0)
+			(at 0.025 3.91 0)
 			(layer "F.Fab")
 			(effects
@@
 		)
 		(property "Value" "PT2399"
-			(at 3.81 20.11 0)
+			(at 3.76 13.28 90)
 			(layer "F.Fab")
 			(effects
@@
 		(embedded_fonts no)
 	)
+	(gr_text "RATE"
+		(at 129.41 123.59 0)
+		(layer "F.SilkS")
+		(effects
+			(font
+				(size 1.5 1.5)
+				(thickness 0.25)
+				(bold yes)
+			)
+		)
+	)
+	(gr_text "IN"
+		(at 128.25 59.5 0)
+		(layer "F.SilkS")
+		(effects
+			(font
+				(size 1.5 1.5)
+				(thickness 0.25)
+				(bold yes)
+			)
+		)
+	)
+	(gr_text "FEED"
+		(at 129.185 108.874001 0)
+		(layer "F.SilkS")
+		(effects
+			(font
+				(size 1.5 1.5)
+				(thickness 0.25)
+				(bold yes)
+			)
+		)
+	)
+	(gr_text "OUT"
+		(at 172.25 59.5 0)
+		(layer "F.SilkS")
+		(effects
+			(font
+				(size 1.5 1.5)
+				(thickness 0.25)
+				(bold yes)
+			)
+		)
+	)
+	(gr_text "DECAY"
+		(at 170.75 108.75 0)
+		(layer "F.SilkS")
+		(effects
+			(font
+				(size 1.5 1.5)
+				(thickness 0.25)
+				(bold yes)
+			)
+		)
+	)
+	(gr_text "DEPTH"
+		(at 170.725 123.515999 0)
+		(layer "F.SilkS")
+		(effects
+			(font
+				(size 1.5 1.5)
+				(thickness 0.25)
+				(bold yes)
+			)
+		)
+	)
 	(segment
 		(start 132.5185 50.601)
@@
 		(width 0.5)
 		(layer "B.Cu")
-		(net 7)
-	)
-	(segment
-		(start 150.3 91.6)
-		(end 146.2 91.6)
-		(width 0.5)
-		(layer "B.Cu")

Commit message: Chorus DRC
Parts:
- added G***: LOGO, HackSynth:Rabbit, B.Cu at (152.2, 95.0)
- added G***: LOGO, HackSynth:Logo - PancakeLegend 10mm Invert, B.Cu at (192.5, 110.2)
- moved G1 90.2 mm to (195.8, 137.2)
- moved G2 39.0 mm to (192.2, 124.5)
Routing:
- net Net-(U4-LPF2-IN): track 30.8 -> 30.0 mm
Other:
- board text added: "CHORUS v1-0 - PancakeLegend 2025"

Commit message: Chorus Backups
Parts:
- removed the G*** at (152.2, 95.0)
- added G***: LOGO, HackSynth:Logo - Rabbit, B.Cu at (149.9, 92.4)
- moved G1 27.3 mm to (205.8, 111.9)
- moved G2 27.2 mm to (199.3, 98.2)
Other:
- board text added: "CHORUS v1-0 PancakeLegend 2025"
- board text removed: "CHORUS v1-0 - PancakeLegend 2025"

Commit message: Chorus Gerbers
Parts:
- removed the G*** at (149.9, 92.4)
- added G***: LOGO, HackSynth:Logo - Rabbit 02, B.Cu at (150.0, 94.2)
