File: KiCAD/LFO/v1-0/LFO.kicad_pcb (KiCad board)
At the start: 2 copper layers, 30 x 100 mm, 16 parts, among them J1 OUT, J2 OUT, J3 Conn_01x03, J4 Conn_01x03, SW1 SW_SPDT, U1 TL072

Commit message: Fixes
Connections:
- C1 pad 1: Net-(U1A--) -> Net-(SW1-A)
- R1 pad 1: Net-(U1A--) -> Net-(R1-Pad1)
- RV1 pad 1: Net-(SW1-A) -> Net-(R1-Pad1)
- RV1 pad 2: Net-(SW1-A) -> Net-(R1-Pad1)
- U1 pad 2: Net-(U1A--) -> Net-(SW1-A)
Routing:
- net Net-(R1-Pad1): track 0.00 -> 38.3 mm, vias 0 -> 1
- net Net-(U1A--): track 18.2 -> 0.00 mm
- net Net-(SW1-A): track 38.1 -> 40.4 mm
Other:
- board text added: "LFO v1-0-1"
- board text added: "PancakeLegend 2026"
- board text removed: "LFO v1-0"
- board text removed: "PancakeLegend 2025"
