File: KiCAD/LFO/v1-1/LFO.kicad_sch (KiCad schematic)
At the start: 22 parts, among them J1 OUT, J2 OUT, J3 Conn_01x03, J4 Conn_01x03, SW1 SW_SPDT, SW2 SW_SPDT, U1 TL072, U2 TL072

Commit message: Fixes
Connections:
- net at RV1.1, RV1.2: now also R1.1; no longer R1.2, SW1.1 (A)
- net at C1.1, U1.2 (-): now also R1.2, SW1.1 (A); no longer R1.1
- net at C2.1, U2.2 (-): now also R5.2, SW2.1 (A); no longer R5.1
- net at RV2.1, RV2.2: now also R5.1; no longer R5.2, SW2.1 (A)
Other:
- moved on the sheet: R1, R5
Changed lines of the file:
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@@
 	(wire
 		(pts
-			(xy 39.37 62.23) (xy 39.37 55.88)
+			(xy 39.37 43.18) (xy 39.37 62.23)
 		)
 		(stroke
@@
 	(wire
 		(pts
-			(xy 39.37 43.18) (xy 59.69 43.18)
+			(xy 39.37 43.18) (xy 41.91 43.18)
 		)
 		(stroke
@@
 	(wire
 		(pts
-			(xy 39.37 43.18) (xy 39.37 48.26)
-		)
-		(stroke
-			(width 0)
-			(type default)
-		)
-	)
-	(wire
-		(pts
 			(xy 39.37 130.81) (xy 48.26 130.81)
 		)
@@
 	(wire
 		(pts
-			(xy 39.37 130.81) (xy 39.37 124.46)
+			(xy 39.37 111.76) (xy 39.37 130.81)
 		)
 		(stroke
@@
 	(wire
 		(pts
-			(xy 39.37 111.76) (xy 59.69 111.76)
+			(xy 39.37 111.76) (xy 41.91 111.76)
 		)
 		(stroke
@@
 	(wire
 		(pts
+			(xy 49.53 111.76) (xy 59.69 111.76)
+		)
+		(stroke
+			(width 0)
+			(type default)
+		)
+	)
+	(wire
+		(pts
 			(xy 59.69 111.76) (xy 62.23 111.76)
 		)
@@
 	(wire
 		(pts
-			(xy 39.37 111.76) (xy 39.37 116.84)
-		)
-		(stroke
-			(width 0)
-			(type default)
-		)
-	)
-	(wire
-		(pts
 			(xy 69.85 43.18) (xy 73.66 43.18)
 		)
@@
 	(wire
 		(pts
+			(xy 49.53 43.18) (xy 59.69 43.18)
+		)
+		(stroke
+			(width 0)
+			(type default)
+		)
+	)
+	(wire
+		(pts
 			(xy 73.66 140.97) (xy 73.66 143.51)
 		)
@@
 	(symbol
 		(lib_id "HackSynth:R")
-		(at 39.37 52.07 180)
+		(at 45.72 43.18 270)
 		(unit 1)
 		(exclude_from_sim no)
@@
 		(dnp no)
 		(property "Reference" "R1"
-			(at 37.338 51.054 0)
+			(at 45.72 36.83 90)
 			(effects
 				(font
 					(size 1.27 1.27)
 				)
-				(justify left)
 			)
 		)
 		(property "Value" "10k"
-			(at 37.338 53.0861 0)
+			(at 45.72 39.37 90)
 			(effects
 				(font
 					(size 1.27 1.27)
 				)
-				(justify left)
 			)
 		)
 		(property "Footprint" "HackSynth:R_Axial_DIN0207_L6.3mm_D2.5mm_P7.62mm_Horizontal"
-			(at 41.148 52.07 90)
+			(at 45.72 41.402 90)
 			(effects
 				(font
@@
 		)
 		(property "Datasheet" "~"
-			(at 39.37 52.07 0)
+			(at 45.72 43.18 0)
 			(effects
 				(font
@@
 		)
 		(property "Description" "Resistor"
-			(at 39.37 52.07 0)
+			(at 45.72 43.18 0)
 			(effects
 				(font
@@
 	(symbol
 		(lib_id "HackSynth:R")
-		(at 39.37 120.65 180)
+		(at 45.72 111.76 270)
 		(unit 1)
 		(exclude_from_sim no)
@@
 		(dnp no)
 		(property "Reference" "R5"
-			(at 37.338 119.634 0)
+			(at 45.72 105.41 90)
 			(effects
 				(font
 					(size 1.27 1.27)
 				)
-				(justify left)
 			)
 		)
 		(property "Value" "10k"
-			(at 37.338 121.6661 0)
+			(at 45.72 107.95 90)
 			(effects
 				(font
 					(size 1.27 1.27)
 				)
-				(justify left)
 			)
 		)
 		(property "Footprint" "HackSynth:R_Axial_DIN0207_L6.3mm_D2.5mm_P7.62mm_Horizontal"
-			(at 41.148 120.65 90)
+			(at 45.72 109.982 90)
 			(effects
 				(font
@@
 		)
 		(property "Datasheet" "~"
-			(at 39.37 120.65 0)
+			(at 45.72 111.76 0)
 			(effects
 				(font
@@
 		)
 		(property "Description" "Resistor"
-			(at 39.37 120.65 0)
+			(at 45.72 111.76 0)
 			(effects
 				(font
