File: KiCAD/LFO/v1-1/LFO.kicad_pcb (KiCad board)
At the start: 2 copper layers, 30 x 100 mm, 23 parts, among them J1 OUT, J2 OUT, J3 Conn_01x03, J4 Conn_01x03, SW1 SW_SPDT, SW2 SW_SPDT, U1 TL072, U2 TL072

Commit message: Fixes
Parts:
- removed Ref**: Val**, HackSynth:CCHS Logo - 10mm
Connections:
- C1 pad 1: Net-(U1A--) -> Net-(SW1-A)
- C2 pad 1: Net-(U2A--) -> Net-(SW2-A)
- R1 pad 1: Net-(U1A--) -> Net-(R1-Pad1)
- R5 pad 1: Net-(U2A--) -> Net-(R5-Pad1)
- RV1 pad 1: Net-(SW1-A) -> Net-(R1-Pad1)
- RV1 pad 2: Net-(SW1-A) -> Net-(R1-Pad1)
- RV2 pad 1: Net-(SW2-A) -> Net-(R5-Pad1)
- RV2 pad 2: Net-(SW2-A) -> Net-(R5-Pad1)
- U1 pad 2: Net-(U1A--) -> Net-(SW1-A)
- U2 pad 2: Net-(U2A--) -> Net-(SW2-A)
Routing:
- net Net-(U1A--): track 41.0 -> 0.00 mm
- net Net-(U2A--): track 40.3 -> 0.00 mm
- net VSS: track 71.4 -> 90.9 mm
- net Net-(R5-Pad1): track 0.00 -> 11.0 mm
- net Net-(R1-Pad1): track 0.00 -> 11.0 mm
- net Net-(SW1-A): track 31.2 -> 41.8 mm
- net Net-(SW2-A): track 31.2 -> 41.8 mm

Commit message: Gerbers - Minor Edits
Parts:
- added Ref**: Val**, HackSynth:CCHS Logo - 10mm, B.Cu at (142.3, 73.5)
