File: KiCAD/VCO/v1-1/VCO.kicad_sch (KiCad schematic)
At the start: 41 parts, among them J1 CV IN 1, J2 CV IN 2, J3 PWM, J4 SAW OUT, J5 PULSE OUT, J6 Conn_01x03_Pin, J7 Conn_01x03_Pin, Q1 NPN, T1 PNP, T2 NPN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

Commit message: Gerbers
Parts:
- D1, D2: value D -> 1N4148
- Q1, T2: value NPN -> BC548 NPN
- RV1: value R_Potentiometer -> 22k
- RV2: value R_Potentiometer_Trim 1k -> 1k Trimpot
- RV3: value PW ADJUST -> 22k
- T1: value PNP -> BC558 PNP
Connections:
- net GND: now also U1.7 (VSS)
- net VSS: now also T1.1 (C); no longer T1.3 (E), U1.7 (VSS)
- net at R10.2, T2.2 (B): now also T1.3 (E); no longer T1.1 (C)
Other:
- note added: "PW ADJUST"
- note removed: "Check Pin Order on Footprint"
- moved on the sheet: U1G
