File: KiCAD/VCO/v1-1/VCO.kicad_pcb (KiCad board)
At the start: 2 copper layers, 50 x 100 mm, 42 parts, among them J1 CV IN 1, J2 CV IN 2, J3 PWM, J4 SAW OUT, J5 PULSE OUT, J6 Conn_01x03_Pin, J7 Conn_01x03_Pin, Q1 NPN, T1 PNP, T2 NPN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

Commit message: Gerbers
Parts:
- added Ref**: Val**, HackSynth:CCHS Logo - 10mm, B.Cu at (89.8, 70.3)
- added Ref**: Val**, HackSynth:PancakeLegend Logo - 10mm, B.Cu at (60.0, 70.4)
- D1, D2: value D -> 1N4148
- Q1, T2: value NPN -> BC548 NPN
- R15: value R -> 680R
- R19: value R -> 22K
- RV1: value R_Potentiometer -> 22k
- RV2: value R_Potentiometer_Trim 1k -> 1k Trimpot
- RV3: value PW ADJUST -> 22k
- T1: value PNP -> BC558 PNP
Connections:
- R10 pad 2: Net-(T1-C) -> Net-(T1-E)
- T1 pad 1: Net-(T1-C) -> VSS
- T1 pad 3: VSS -> Net-(T1-E)
- T2 pad 2: Net-(T1-C) -> Net-(T1-E)
- U1 pad 7: VSS -> GND
Routing:
- net Net-(T1-E): track 0.00 -> 26.1 mm
- net Net-(T1-C): track 22.1 -> 0.00 mm
- net Net-(R1-Pad1): track 19.3 -> 21.4 mm
- net Net-(R17-Pad2): track 38.7 -> 40.6 mm
- net Net-(T1-B): track 34.6 -> 36.3 mm, vias 0 -> 1
- net Net-(Q1-E): track 63.2 -> 61.6 mm
- net VSS: track 85.1 -> 83.9 mm
- net Net-(D2-K): track 69.8 -> 70.7 mm, vias 0 -> 1
- net Net-(R2-Pad2): track 17.6 -> 18.1 mm
- net GND: track 3.50 -> 3.00 mm
Other:
- board text added: "VCO v1-1 - Dfatpnuk / PancakeLegend 2026"

Commit message: Gerbers - Minor Edits
Parts:
- moved Ref** 0.30 mm to (60.0, 70.1)
- moved Ref** 0.30 mm to (89.8, 70.0)
Other:
- board text added: "VCO"
Changed lines of the file:
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@@
 	(footprint "HackSynth:CCHS Logo - 10mm"
 		(layer "B.Cu")
-		(at 89.8 70.3 180)
+		(at 89.8 70 180)
 		(property "Reference" "Ref**"
 			(at 0 0 0)
@@
 	(footprint "HackSynth:PancakeLegend Logo - 10mm"
 		(layer "B.Cu")
-		(at 60 70.4 180)
+		(at 60 70.1 180)
 		(property "Reference" "Ref**"
 			(at 0 0 0)
@@
 		(embedded_fonts no)
 	)
+	(gr_line
+		(start 80.500001 68.699998)
+		(end 80.500001 71.699997)
+		(stroke
+			(width 0.5)
+			(type solid)
+		)
+		(layer "B.SilkS")
+	)
+	(gr_line
+		(start 79.000001 73.2)
+		(end 70.999998 73.2)
+		(stroke
+			(width 0.5)
+			(type solid)
+		)
+		(layer "B.SilkS")
+	)
+	(gr_arc
+		(start 79.000002 67.199997)
+		(mid 80.060662 67.639338)
+		(end 80.500001 68.699998)
+		(stroke
+			(width 0.5)
+			(type solid)
+		)
+		(layer "B.SilkS")
+	)
+	(gr_arc
+		(start 80.500001 71.7)
+		(mid 80.060661 72.76066)
+		(end 79.000002 73.200001)
+		(stroke
+			(width 0.5)
+			(type solid)
+		)
+		(layer "B.SilkS")
+	)
+	(gr_line
+		(start 69.500001 68.7)
+		(end 69.500001 71.699999)
+		(stroke
+			(width 0.5)
+			(type solid)
+		)
+		(layer "B.SilkS")
+	)
+	(gr_arc
+		(start 70.999998 73.2)
+		(mid 69.939339 72.760659)
+		(end 69.499999 71.7)
+		(stroke
+			(width 0.5)
+			(type solid)
+		)
+		(layer "B.SilkS")
+	)
+	(gr_arc
+		(start 69.500001 68.7)
+		(mid 69.939341 67.639341)
+		(end 71 67.199999)
+		(stroke
+			(width 0.5)
+			(type solid)
+		)
+		(layer "B.SilkS")
+	)
+	(gr_line
+		(start 78.999999 67.199998)
+		(end 71 67.199999)
+		(stroke
+			(width 0.5)
+			(type solid)
+		)
+		(layer "B.SilkS")
+	)
 	(gr_text "IN 2"
 		(at 60 71 0)
@@
 	)
 	(gr_text "VCO v1-1 - Dfatpnuk / PancakeLegend 2026"
-		(at 96 53.4 0)
+		(at 75.1 131.25 0)
 		(layer "B.SilkS")
 		(effects
@@
 				(thickness 0.15)
 			)
-			(justify left bottom mirror)
+			(justify mirror)
+		)
+	)
+	(gr_text "VCO"
+		(at 75 70.4 0)
+		(layer "B.SilkS")
+		(effects
+			(font
+				(size 3 3)
+				(thickness 0.5)
+				(bold yes)
+			)
+			(justify mirror)
 		)
 	)
@@
 		)
 	)
+	(group ""
+		(members "169c76da-6227-4311-bb50-b279aba2962e" "19239882-9ef9-4554-bdf6-0972030d447c"
+			"196c336a-56b8-4261-90cb-e83e8f6fe0b1" "54609670-d5b0-4a71-89d8-4731b9f57049"
+			"791d8a8b-b674-458c-a312-2b7d63c2b197" "80884f73-dd9b-43b8-bc6f-e9734f687da7"
+			"96a65055-7344-4382-a680-1624404822ec" "d0aeac7a-8426-49e8-a1fc-1eea3f70c9e1"
+			"fc37200a-bd09-49b1-a2a7-5d3c20eeec03"
+		)
+	)
